File: hardware/src/TmpUsb-A [B].kicad_pcb (KiCad board)
At the start: 2 copper layers, 25 x 17 mm, 17 parts, among them P1 48037-2200, U1 PIC18F26J50

Commit message: Replaced ferrite bead footprint
Parts:
- L1: footprint Medo64-SMD:L (0805) -> Medo64-SMD:L Ferrite (0805)
Changed lines of the file:
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@@
     )
   )
-  (footprint "Medo64-SMD:L (0805)" (layer "F.Cu")
+  (footprint "Medo64-SMD:L Ferrite (0805)" (layer "F.Cu")
     (at 25.9 34.9 -90)
     (descr "RESC2013X70N")
