File: hardware/src/TmpUsb-A.kicad_pcb (KiCad board)
At the start: 2 copper layers, 25 x 17 mm, 17 parts, among them P1 48037-2200, U1 PIC18F26J50

Commit message: Updated ICSP footprint
Other:
- board text added: "TmpUsb:A B"
- board text removed: "TmpUsb-A B"
Changed lines of the file:
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@@
         (effects (font (size 0.7 0.6) (thickness 0.1) bold) (justify top mirror))
-    )
-    (fp_text user "PGD" (at 3.81 1.07 unlocked) (layer "User.7")
-        (effects (font (size 0.13 0.07) (thickness 0.01)) (justify top))
-    )
-    (fp_text user "Vdd" (at -3.81 1.07 unlocked) (layer "User.7")
-        (effects (font (size 0.13 0.07) (thickness 0.014) bold) (justify top))
     )
     (fp_text user "Vpp" (at -6.35 1.07 unlocked) (layer "User.7")
@@
     (fp_text user "PGC" (at 1.27 1.07 unlocked) (layer "User.7")
         (effects (font (size 0.13 0.07) (thickness 0.01)) (justify top))
+    )
+    (fp_text user "PGD" (at 3.81 1.07 unlocked) (layer "User.7")
+        (effects (font (size 0.13 0.07) (thickness 0.01)) (justify top))
+    )
+    (fp_text user "Vdd" (at -3.81 1.07 unlocked) (layer "User.7")
+        (effects (font (size 0.13 0.07) (thickness 0.014) bold) (justify top))
     )
     (fp_rect (start -7.62 1.27) (end 7.62 -1.27)
@@
   (gr_line (start 22 20) (end 41 20)
     (stroke (width 0.05) (type default)) (layer "Edge.Cuts"))
-  (gr_text "TmpUsb-A B" (at 42.352 36.238) (layer "B.SilkS")
+  (gr_text "TmpUsb:A B" (at 42.352 36.238) (layer "B.SilkS")
     (effects (font (size 1 1) (thickness 0.15)) (justify left bottom mirror))
   )
