File: hardware/src/TmpUsb'A.kicad_pcb (KiCad board)
At the start: 2 copper layers, 25 x 17 mm, 17 parts, among them P1 48037-2200, U1 PIC18F26J50

Commit message: Updated footprints
Parts:
- ?: footprint Medo64:ICSP PIC Pogo' (5w) -> Medo64:ICSP PIC Pogo SS (5w)
- moved ? 7.07 mm to (27.7, 21.5)
- moved C1 7.07 mm to (29.7, 29.9)
- moved R4 7.07 mm to (35.1, 30.7)
- moved C2 7.07 mm to (23.8, 16.3)
- moved C3 7.07 mm to (23.1, 29.9)
- moved C4 7.07 mm to (32.0, 29.9)
- moved C5 7.07 mm to (28.0, 16.3)
- moved C6 7.07 mm to (35.1, 28.4)
- moved DS1 7.07 mm to (34.6, 23.5)
- moved L1 7.07 mm to (20.9, 29.9)
- moved P1 7.07 mm to (17.8, 23.5)
- moved R1 7.07 mm to (35.1, 16.3)
- moved R2 7.07 mm to (35.1, 26.1)
- moved R3 7.07 mm to (35.1, 18.6)
- moved U1 7.07 mm to (27.5, 22.4)
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
Commit message: Rotated LED around and minor component updates
Parts:
- moved DS1 0.20 mm to (34.8, 23.5), turned to 0 degrees
Connections:
- DS1 pad 1: LED' -> GND
- DS1 pad 2: GND -> LED'
Other:
- board text added: "ACT"
Changed lines of the file:
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@@
   (footprint "Medo64:R (0805)" (layer "F.Cu")
     (at 35.1 30.7 180)
-    (descr "RESC2013X70N")
+    (tags "RESC2013X70N")
     (attr smd)
     (fp_text reference "R4" (at 0 -1.6 180 unlocked) (layer "F.SilkS") hide
@@
   (footprint "Medo64:R (0805)" (layer "F.Cu")
     (at 35.1 16.3)
-    (descr "RESC2013X70N")
+    (tags "RESC2013X70N")
     (attr smd)
     (fp_text reference "R1" (at 0 -1.6 unlocked) (layer "F.SilkS") hide
         (effects (font (size 0.8 0.6) (thickness 0.15)))
     )
-    (fp_text value "1K" (at -2.4 0 unlocked) (layer "F.SilkS")
+    (fp_text value "1K" (at 2.25 0.6 -90 unlocked) (layer "F.SilkS")
         (effects (font (size 0.8 0.6) (thickness 0.15)))
     )
@@
   )
   (footprint "Medo64:DS (0805)" (layer "F.Cu")
-    (at 34.6 23.5 180)
+    (at 34.8 23.5)
     (descr "LEDC2013X120N")
     (attr smd)
-    (fp_text reference "DS1" (at 0 -1.5 180 unlocked) (layer "F.Fab")
-        (effects (font (size 0.8 0.6) (thickness 0.15) bold))
-    )
-    (fp_text value "ACT" (at 0 1.6 unlocked) (layer "F.SilkS")
+    (fp_text reference "DS1" (at 0 -1.5 unlocked) (layer "F.Fab") hide
+        (effects (font (size 0.8 0.6) (thickness 0.15) bold))
+    )
+    (fp_text value "ACT" (at 0.1 -1.6 unlocked) (layer "F.SilkS") hide
         (effects (font (size 0.8 0.6) (thickness 0.15) bold))
     )
@@
     (fp_rect (start -1 -0.625) (end 1 0.625)
       (stroke (width 0.01) (type dash_dot)) (fill none) (layer "F.Fab"))
-    (pad "1" smd roundrect (at -0.9 0 180) (size 1 1.4) (layers "F.Cu" "F.Paste" "F.Mask") (roundrect_rratio 0.25)
+    (pad "1" smd roundrect (at -0.9 0) (size 1 1.4) (layers "F.Cu" "F.Paste" "F.Mask") (roundrect_rratio 0.25)
       (chamfer_ratio 0.2) (chamfer top_left bottom_left)
+      (net 3 "GND") (thermal_bridge_angle 45))
+    (pad "2" smd roundrect (at 0.9 0) (size 1 1.4) (layers "F.Cu" "F.Paste" "F.Mask") (roundrect_rratio 0.25)
       (net 9 "LED'") (thermal_bridge_angle 45))
-    (pad "2" smd roundrect (at 0.9 0 180) (size 1 1.4) (layers "F.Cu" "F.Paste" "F.Mask") (roundrect_rratio 0.25)
-      (net 3 "GND") (thermal_bridge_angle 45))
     (model ":KICAD7_3DMODEL_DIR:LED_SMD.3dshapes/LED_0805_2012Metric.step"
       (offset (xyz 0 0 0))
@@
         (effects (font (size 0.8 0.6) (thickness 0.15)))
     )
-    (fp_text user "D+" (at -1 -1.5 -90 unlocked) (layer "Cmts.User")
+    (fp_text user "D-" (at 1 -1.5 -90 unlocked) (layer "Cmts.User" knockout)
         (effects (font (size 0.13 0.07) (thickness 0.01)) (justify top))
     )
-    (fp_text user "Vbus" (at 3.5 -1.5 -90 unlocked) (layer "Cmts.User")
+    (fp_text user "GND" (at -3.5 -1.5 -90 unlocked) (layer "Cmts.User" knockout)
         (effects (font (size 0.13 0.07) (thickness 0.01) bold) (justify top))
     )
-    (fp_text user "GND" (at -3.5 -1.5 -90 unlocked) (layer "Cmts.User")
+    (fp_text user "Vbus" (at 3.5 -1.5 -90 unlocked) (layer "Cmts.User" knockout)
         (effects (font (size 0.13 0.07) (thickness 0.01) bold) (justify top))
     )
-    (fp_text user "D-" (at 1 -1.5 -90 unlocked) (layer "Cmts.User")
+    (fp_text user "D+" (at -1 -1.5 -90 unlocked) (layer "Cmts.User" knockout)
         (effects (font (size 0.13 0.07) (thickness 0.01)) (justify top))
     )
@@
     (pad "4" smd roundrect (at -3.5 -2.6 270) (size 1.2 2) (layers "F.Cu" "F.Paste" "F.Mask") (roundrect_rratio 0.25)
       (net 3 "GND") (thermal_bridge_angle 45))
-    (pad "5" thru_hole oval (at -5.85 0 270) (size 1.3 3.2) (drill oval 0.7 2.5) (layers "*.Cu" "*.Mask" "F.Paste")
-      (thermal_bridge_angle 45))
-    (pad "5" thru_hole oval (at 5.85 0 270) (size 1.3 3.2) (drill oval 0.7 2.5) (layers "*.Cu" "*.Mask" "F.Paste")
+    (pad "S" thru_hole oval (at -5.85 0 270) (size 1.3 3.2) (drill oval 0.7 2.5) (layers "*.Cu" "*.Mask" "F.Paste")
+      (thermal_bridge_angle 45))
+    (pad "S" thru_hole oval (at 5.85 0 270) (size 1.3 3.2) (drill oval 0.7 2.5) (layers "*.Cu" "*.Mask" "F.Paste")
       (thermal_bridge_angle 45))
     (model "../../3dmodels/Medo64-SMD.3dshapes/480372200.step"
@@
   (footprint "Medo64:R (0805)" (layer "F.Cu")
     (at 35.1 18.6)
-    (descr "RESC2013X70N")
+    (tags "RESC2013X70N")
     (attr smd)
     (fp_text reference "R3" (at 0 -1.6 unlocked) (layer "F.SilkS") hide
         (effects (font (size 0.8 0.6) (thickness 0.15)))
     )
-    (fp_text value "10K" (at 0.95 1.7 unlocked) (layer "F.SilkS")
+    (fp_text value "10K" (at 2.25 0.1 -90 unlocked) (layer "F.SilkS")
         (effects (font (size 0.8 0.6) (thickness 0.15)))
     )
@@
   (footprint "Medo64:R (0805)" (layer "F.Cu")
     (at 35.1 26.1)
-    (descr "RESC2013X70N")
+    (tags "RESC2013X70N")
     (attr smd)
     (fp_text reference "R2" (at 0 -1.6 unlocked) (layer "F.SilkS") hide
@@
     (effects (font (size 1 1) (thickness 0.15)) (justify left bottom mirror))
   )
+  (gr_text "ACT" (at 34 22.3) (layer "F.SilkS" knockout)
+    (effects (font (size 1 0.8) (thickness 0.2) bold) (justify left bottom))
+  )
   (segment (start 23.925 24.615) (end 22.801 23.491) (width 0.4) (layer "F.Cu") (net 1))
   (segment (start 22.801 23.491) (end 21.765 23.491) (width 0.4) (layer "F.Cu") (net 1))
@@
   (segment (start 23.1 29) (end 26.28 29) (width 0.2) (layer "F.Cu") (net 3))
   (segment (start 26.28 29) (end 26.28 30.85) (width 0.2) (layer "F.Cu") (net 3))
-  (segment (start 33.7 23.5) (end 35.1 24.9) (width 0.2) (layer "F.Cu") (net 3))
   (segment (start 27.192 20.316) (end 26.991 20.316) (width 0.2) (layer "F.Cu") (net 3))
   (segment (start 27.175 20.299) (end 27.192 20.316) (width 0.2) (layer "F.Cu") (net 3))
+  (segment (start 33.9 23.5) (end 35.1 24.7) (width 0.2) (layer "F.Cu") (net 3))
   (segment (start 27.175 18.9) (end 27.175 20.299) (width 0.2) (layer "F.Cu") (net 3))
   (segment (start 27.55 30.85) (end 29.65 30.85) (width 0.2) (layer "F.Cu") (net 3))
@@
   (segment (start 22.4 20) (end 20.3 20) (width 0.2) (layer "F.Cu") (net 3))
   (segment (start 25.875 25.9) (end 25.875 22.522) (width 0.2) (layer "F.Cu") (net 3))
+  (segment (start 35.1 24.7) (end 35.1 27.5) (width 0.2) (layer "F.Cu") (net 3))
   (segment (start 27.1 16.3) (end 24.7 16.3) (width 0.2) (layer "F.Cu") (net 3))
-  (segment (start 35.1 24.9) (end 35.1 27.5) (width 0.2) (layer "F.Cu") (net 3))
   (segment (start 26.991 20.316) (end 22.716 20.316) (width 0.2) (layer "F.Cu") (net 3))
   (segment (start 27.7 20.6) (end 27.416 20.316) (width 0.2) (layer "F.Cu") (net 3))
@@
   (segment (start 31.075 18.9) (end 31.075 17.625) (width 0.2) (layer "F.Cu") (net 8))
   (segment (start 31.075 17.625) (end 32.4 16.3) (width 0.2) (layer "F.Cu") (net 8))
-  (segment (start 37 21.809) (end 37 17.25) (width 0.2) (layer "F.Cu") (net 9))
-  (segment (start 35.5 23.309) (end 37 21.809) (width 0.2) (layer "F.Cu") (net 9))
+  (segment (start 36.607928 22.392072) (end 36.656054 22.325832) (width 0.2) (layer "F.Cu") (net 9))
+  (segment (start 36.910733 22.089267) (end 37 22) (width 0.2) (layer "F.Cu") (net 9))
+  (segment (start 37 22) (end 37 17.25) (width 0.2) (layer "F.Cu") (net 9))
+  (segment (start 36.887309 22.104729) (end 36.910733 22.089267) (width 0.2) (layer "F.Cu") (net 9))
+  (segment (start 35.7 23.3) (end 36.607928 22.392072) (width 0.2) (layer "F.Cu") (net 9))
   (segment (start 37 17.25) (end 36.05 16.3) (width 0.2) (layer "F.Cu") (net 9))
+  (segment (start 36.656054 22.325832) (end 36.887309 22.104729) (width 0.2) (layer "F.Cu") (net 9))
   (segment (start 20.3 27) (end 20.3 28.65) (width 0.2) (layer "F.Cu") (net 10))
   (segment (start 20.3 28.65) (end 20.8 29.15) (width 0.2) (layer "F.Cu") (net 10))

Commit message: Moving silkscreen around
Routing:
- net GND: track 47.5 -> 49.2 mm
Changed lines of the file:
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@@
         (effects (font (size 0.8 0.6) (thickness 0.15) bold))
     )
-    (fp_text value "10u" (at -2.25 2.65 270 unlocked) (layer "F.SilkS")
+    (fp_text value "10u" (at -2.25 1.2 270 unlocked) (layer "F.SilkS")
         (effects (font (size 0.8 0.6) (thickness 0.15) bold))
     )
@@
         (effects (font (size 0.8 0.6) (thickness 0.15)))
     )
-    (fp_text value "1K" (at 2.25 1.35 -90 unlocked) (layer "F.SilkS")
+    (fp_text value "1K" (at 2.25 -0.65 -90 unlocked) (layer "F.SilkS")
         (effects (font (size 0.8 0.6) (thickness 0.15)))
     )
@@
   (segment (start 22.536 24.126) (end 23.275 24.865) (width 0.4) (layer "F.Cu") (net 2))
   (segment (start 32 30.8) (end 34.05 30.8) (width 0.2) (layer "F.Cu") (net 3))
-  (segment (start 27.7 21.459) (end 27.7 20.6) (width 0.2) (layer "F.Cu") (net 3))
-  (segment (start 27.416 20.316) (end 27.192 20.316) (width 0.2) (layer "F.Cu") (net 3))
+  (segment (start 27.7 21.459) (end 27.7 20.6) (width 0.25) (layer "F.Cu") (net 3))
+  (segment (start 27.416 20.316) (end 27.192 20.316) (width 0.25) (layer "F.Cu") (net 3))
   (segment (start 27.175 18.5) (end 27.175 16.375) (width 0.2) (layer "F.Cu") (net 3))
-  (segment (start 22.716 20.316) (end 22.4 20) (width 0.2) (layer "F.Cu") (net 3))
+  (segment (start 22.716 20.316) (end 22.4 20) (width 0.25) (layer "F.Cu") (net 3))
   (segment (start 26.28 30.85) (end 27.55 30.85) (width 0.2) (layer "F.Cu") (net 3))
+  (segment (start 33.9 23.5) (end 26.45 23.5) (width 0.25) (layer "F.Cu") (net 3))
+  (segment (start 25.875 25.9) (end 25.875 24.075) (width 0.25) (layer "F.Cu") (net 3))
   (segment (start 25.875 29) (end 23.1 29) (width 0.2) (layer "F.Cu") (net 3))
   (segment (start 25.875 25.9) (end 25.875 29) (width 0.2) (layer "F.Cu") (net 3))
   (segment (start 23.1 29) (end 26.28 29) (width 0.2) (layer "F.Cu") (net 3))
+  (segment (start 25.875 24.075) (end 26.25 23.7) (width 0.25) (layer "F.Cu") (net 3))
   (segment (start 26.28 29) (end 26.28 30.85) (width 0.2) (layer "F.Cu") (net 3))
-  (segment (start 27.192 20.316) (end 26.991 20.316) (width 0.2) (layer "F.Cu") (net 3))
-  (segment (start 27.175 20.299) (end 27.192 20.316) (width 0.2) (layer "F.Cu") (net 3))
-  (segment (start 33.9 23.5) (end 35.1 24.7) (width 0.2) (layer "F.Cu") (net 3))
-  (segment (start 27.175 18.9) (end 27.175 20.299) (width 0.2) (layer "F.Cu") (net 3))
+  (segment (start 27.192 20.316) (end 26.991 20.316) (width 0.25) (layer "F.Cu") (net 3))
+  (segment (start 27.175 20.299) (end 27.192 20.316) (width 0.25) (layer "F.Cu") (net 3))
+  (segment (start 26.416637 23.466637) (end 26.45 23.5) (width 0.25) (layer "F.Cu") (net 3))
+  (segment (start 27.175 18.9) (end 27.175 20.299) (width 0.25) (layer "F.Cu") (net 3))
   (segment (start 27.55 30.85) (end 29.65 30.85) (width 0.2) (layer "F.Cu") (net 3))
   (segment (start 29.7 30.8) (end 32 30.8) (width 0.2) (layer "F.Cu") (net 3))
-  (segment (start 35.1 27.5) (end 34.2 28.4) (width 0.2) (layer "F.Cu") (net 3))
   (segment (start 34.2 28.4) (end 34.2 30.65) (width 0.2) (layer "F.Cu") (net 3))
-  (segment (start 26.416637 21.980363) (end 26.416637 20.316) (width 0.2) (layer "F.Cu") (net 3))
-  (segment (start 25.875 22.522) (end 26.416637 21.980363) (width 0.2) (layer "F.Cu") (net 3))
-  (segment (start 22.4 20) (end 20.3 20) (width 0.2) (layer "F.Cu") (net 3))
-  (segment (start 25.875 25.9) (end 25.875 22.522) (width 0.2) (layer "F.Cu") (net 3))
-  (segment (start 35.1 24.7) (end 35.1 27.5) (width 0.2) (layer "F.Cu") (net 3))
+  (segment (start 22.4 20) (end 20.3 20) (width 0.25) (layer "F.Cu") (net 3))
+  (segment (start 26.45 23.5) (end 26.25 23.7) (width 0.25) (layer "F.Cu") (net 3))
+  (segment (start 26.416637 20.316) (end 26.416637 23.466637) (width 0.25) (layer "F.Cu") (net 3))
   (segment (start 27.1 16.3) (end 24.7 16.3) (width 0.2) (layer "F.Cu") (net 3))
-  (segment (start 26.991 20.316) (end 22.716 20.316) (width 0.2) (layer "F.Cu") (net 3))
-  (segment (start 27.7 20.6) (end 27.416 20.316) (width 0.2) (layer "F.Cu") (net 3))
-  (segment (start 26.416637 20.316) (end 26.991 20.316) (width 0.2) (layer "F.Cu") (net 3))
+  (segment (start 26.991 20.316) (end 22.716 20.316) (width 0.25) (layer "F.Cu") (net 3))
+  (segment (start 27.7 20.6) (end 27.416 20.316) (width 0.25) (layer "F.Cu") (net 3))
+  (segment (start 26.991 20.316) (end 26.416637 20.316) (width 0.25) (layer "F.Cu") (net 3))
   (segment (start 36 28.4) (end 36 26.15) (width 0.3) (layer "F.Cu") (net 4))
   (segment (start 36 27.2) (end 36 26.15) (width 0.3) (layer "F.Cu") (net 4))
