File: hardware/src/TmpUsb'A.kicad_pcb (KiCad board)
At the start: 2 copper layers, 25 x 17 mm, 17 parts, among them J1 48037-2200, U1 PIC18F26J50

Commit message: Renamed V+ nets
Connections:
- net +3.3V renamed 3V3
- net +5V renamed 5V
- net VCAP renamed 3V3_VCAP
- net VCC renamed 5V_USB
